Commit message: support gripper control with seperate left right joint

File: ros2_ws/src/my_ur3/urdf/gripper.xacro (robot description, xacro)
@@ -124,9 +124,4 @@
         effort="50"
         velocity="0.2"/>
-      <!-- Left finger follows right finger -->
-      <mimic
-        joint="right_finger_joint"
-        multiplier="1.0"
-        offset="0.0"/>
     </joint>
   </xacro:macro>

File: ros2_ws/src/my_ur3/urdf/my_ur3_ros2_control.xacro (robot description, xacro)
@@ -13,5 +13,7 @@
                    wrist_1_joint=-1.57,
                    wrist_2_joint=0.0,
-                   wrist_3_joint=0.0
+                   wrist_3_joint=0.0,
+                   right_finger_joint=0.04,
+                   left_finger_joint=0.04
                  )}
                ">
@@ -34,4 +36,11 @@
       <!-- ================================================== -->
       <joint name="right_finger_joint">
+        <param name="initial_value">${initial_positions['right_finger_joint']}</param>
+        <command_interface name="position"/>
+        <state_interface name="position"/>
+        <state_interface name="velocity"/>
+      </joint>
+      <joint name="left_finger_joint">
+        <param name="initial_value">${initial_positions['left_finger_joint']}</param>
         <command_interface name="position"/>
         <state_interface name="position"/>
