Commit message: add comment

File: ros2_ws/src/robot_gripper/urdf/robot_gripper.urdf.xacro (robot description, xacro)
@@ -1,7 +1,14 @@
+<!-- ===================================================== -->
+<!-- Combine UR3 and Robotiq Gripper -->
+<!-- ===================================================== -->
 <?xml version="1.0"?>
 <robot xmlns:xacro="http://ros.org/wiki/xacro" name="robot gripper">
+    <!-- ===================================================== -->
+    <!-- Include UR3 macros -->
+    <!-- ===================================================== -->
     <xacro:include filename="$(find ur_description)/urdf/ur_macro.xacro" />
-    <xacro:include filename="$(find robot_gripper)/urdf/robotiq_arg2f_85_model_macro.xacro" />
-      <!-- UR3 parameters -->
+    <!-- ===================================================== -->
+    <!-- UR3 parameters -->
+    <!-- ===================================================== -->
     <xacro:arg name="tf_prefix" default=""/>
     <xacro:arg
@@ -21,4 +28,7 @@
     <!-- ===================================================== -->
     <link name="world"/>
+    <!-- ===================================================== -->
+    <!-- UR3, link to world -->
+    <!-- ===================================================== -->
     <xacro:ur_robot
         name="ur3"
@@ -36,16 +46,23 @@
             xyz="0 0 0"
             rpy="0 0 0"/>
-  </xacro:ur_robot>
-  <xacro:robotiq_arg2f_85 prefix=""/>
-  <!-- ===================================================== -->
-  <!-- Attach gripper to UR3 tool0 -->
-  <!-- ===================================================== -->
-  <joint name="gripper_to_robot" type="fixed">
-    <parent link="tool0"/>
-    <child link="robotiq_arg2f_base_link"/>
-    <!-- Adjust this after looking at the model -->
-    <origin
-      xyz="0 0 0"
-      rpy="0 0 0"/>
-  </joint>
+    </xacro:ur_robot>
+    <!-- ===================================================== -->
+    <!-- Include Robotiq 2F-85 macros -->
+    <!-- ===================================================== -->
+    <xacro:include filename="$(find robot_gripper)/urdf/robotiq_arg2f_85_model_macro.xacro" />
+    <!-- ===================================================== -->
+    <!-- Robotiq 2F-85 -->
+    <!-- ===================================================== -->
+    <xacro:robotiq_arg2f_85 prefix=""/>
+    <!-- ===================================================== -->
+    <!-- Attach gripper to UR3 tool0 -->
+    <!-- ===================================================== -->
+    <joint name="gripper_to_robot" type="fixed">
+        <parent link="tool0"/>
+        <child link="robotiq_arg2f_base_link"/>
+        <!-- Adjust this after looking at the model -->
+        <origin
+        xyz="0 0 0"
+        rpy="0 0 0"/>
+    </joint>
 </robot>

Commit message: change robotiq ros2 model

File: ros2_ws/src/robot_gripper/urdf/robot_gripper.urdf.xacro (robot description, xacro)
@@ -1,7 +1,7 @@
-<!-- ===================================================== -->
-<!-- Combine UR3 and Robotiq Gripper -->
-<!-- ===================================================== -->
 <?xml version="1.0"?>
 <robot xmlns:xacro="http://ros.org/wiki/xacro" name="robot gripper">
+    <!-- ===================================================== -->
+    <!-- Combine UR3 and Robotiq Gripper -->
+    <!-- ===================================================== -->
     <!-- ===================================================== -->
     <!-- Include UR3 macros -->
@@ -50,19 +50,14 @@
     <!-- Include Robotiq 2F-85 macros -->
     <!-- ===================================================== -->
-    <xacro:include filename="$(find robot_gripper)/urdf/robotiq_arg2f_85_model_macro.xacro" />
+    <xacro:include filename="$(find robot_gripper)/urdf/robotiq_2f_85_macro.urdf.xacro" />
     <!-- ===================================================== -->
     <!-- Robotiq 2F-85 -->
     <!-- ===================================================== -->
-    <xacro:robotiq_arg2f_85 prefix=""/>
-    <!-- ===================================================== -->
-    <!-- Attach gripper to UR3 tool0 -->
-    <!-- ===================================================== -->
-    <joint name="gripper_to_robot" type="fixed">
-        <parent link="tool0"/>
-        <child link="robotiq_arg2f_base_link"/>
-        <!-- Adjust this after looking at the model -->
-        <origin
-        xyz="0 0 0"
-        rpy="0 0 0"/>
-    </joint>
+    <xacro:robotiq_gripper
+        name="RobotiqGripper"
+        prefix=""
+        parent="tool0"
+        sim_gazebo="true">
+        <origin xyz="0 0 0" rpy="0 0 0"/>
+    </xacro:robotiq_gripper>
 </robot>

File: ros2_ws/src/robot_gripper/urdf/robot_gripper_final.urdf (robot description, URDF)
Before this commit: robot robot gripper, 24 links, 23 joints
Links:
- removed link left_inner_finger
- removed link left_inner_finger_pad
- removed link left_inner_knuckle
- removed link left_outer_finger
- removed link left_outer_knuckle
- removed link right_inner_finger
- removed link right_inner_finger_pad
- removed link right_inner_knuckle
- removed link right_outer_finger
- removed link right_outer_knuckle
- removed link robotiq_arg2f_base_link
- added link robotiq_85_base_link, mass 6.6320197e-01; collision mesh filename=package://robotiq_description/meshes/collision/2f_85/roboti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; visual mesh filename=package://robotiq_description/meshes/visual/2f_85/robotiq_b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
- added link robotiq_85_left_finger_link, mass 4.260376752e-02; collision mesh filename=package://robotiq_description/meshes/collision/2f_85/left_f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; visual mesh filename=package://robotiq_description/meshes/visual/2f_85/left_fing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
- added link robotiq_85_left_finger_tip_link, mass 4.268588744e-02; collision mesh filename=package://robotiq_description/meshes/collision/2f_85/left_f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; visual mesh filename=package://robotiq_description/meshes/visual/2f_85/left_fing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
- added link robotiq_85_left_inner_knuckle_link, mass 2.969376448e-02; collision mesh filename=package://robotiq_description/meshes/collision/2f_85/left_i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; visual mesh filename=package://robotiq_description/meshes/visual/2f_85/left_inne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
- added link robotiq_85_left_knuckle_link, mass 1.384773208e-02; collision mesh filename=package://robotiq_description/meshes/collision/2f_85/left_k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; visual mesh filename=package://robotiq_description/meshes/visual/2f_85/left_knuc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
- added link robotiq_85_right_finger_link, mass 4.260376752000000e-02; collision mesh filename=package://robotiq_description/meshes/collision/2f_85/right_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; visual mesh filename=package://robotiq_description/meshes/visual/2f_85/right_fin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
- added link robotiq_85_right_finger_tip_link, mass 4.268588744e-02; collision mesh filename=package://robotiq_description/meshes/collision/2f_85/right_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; visual mesh filename=package://robotiq_description/meshes/visual/2f_85/right_fin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
- added link robotiq_85_right_inner_knuckle_link, mass 2.969376448e-02; collision mesh filename=package://robotiq_description/meshes/collision/2f_85/right_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; visual mesh filename=package://robotiq_description/meshes/visual/2f_85/right_inn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
- added link robotiq_85_right_knuckle_link, mass 1.384773208e-02; collision mesh filename=package://robotiq_description/meshes/collision/2f_85/right_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; visual mesh filename=package://robotiq_description/meshes/visual/2f_85/right_knu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
Joints:
- removed joint finger_joint
- removed joint gripper_to_robot
- removed joint left_inner_finger_joint
- removed joint left_inner_finger_pad_joint
- removed joint left_inner_knuckle_joint
- removed joint left_outer_finger_joint
- removed joint right_inner_finger_joint
- removed joint right_inner_finger_pad_joint
- removed joint right_inner_knuckle_joint
- removed joint right_outer_finger_joint
- removed joint right_outer_knuckle_joint
- added joint robotiq_85_base_joint: type fixed, parent tool0, child robotiq_85_base_link, origin xyz=0 0 0 rpy=0 0 0
- added joint robotiq_85_left_finger_joint: type fixed, parent robotiq_85_left_knuckle_link, child robotiq_85_left_finger_link, origin xyz=0.03152616 0.0 -0.00376347 rpy=0 0 0
- added joint robotiq_85_left_finger_tip_joint: type revolute, parent robotiq_85_left_finger_link, child robotiq_85_left_finger_tip_link, origin xyz=0.00563134 0.0 0.04718515 rpy=0 0 0, axis 0 -1 0, limit lower=-0.8 upper=0.0 effort=50 velocity=0.5, mimic joint=robotiq_85_left_knuckle_joint multiplier=-1
- added joint robotiq_85_left_inner_knuckle_joint: type revolute, parent robotiq_85_base_link, child robotiq_85_left_inner_knuckle_link, origin xyz=0.0127 0.0 0.06142 rpy=0 0 0, axis 0 -1 0, limit lower=0.0 upper=0.8 effort=50 velocity=0.5, mimic joint=robotiq_85_left_knuckle_joint
- added joint robotiq_85_left_knuckle_joint: type revolute, parent robotiq_85_base_link, child robotiq_85_left_knuckle_link, origin xyz=0.03060114 0.0 0.05490452 rpy=0 0 0, axis 0 -1 0, limit lower=0.0 upper=0.8 effort=50 velocity=0.5
- added joint robotiq_85_right_finger_joint: type fixed, parent robotiq_85_right_knuckle_link, child robotiq_85_right_finger_link, origin xyz=-0.03152616 0.0 -0.00376347 rpy=0 0 0
- added joint robotiq_85_right_finger_tip_joint: type revolute, parent robotiq_85_right_finger_link, child robotiq_85_right_finger_tip_link, origin xyz=-0.00563134 0.0 0.04718515 rpy=0 0 0, axis 0 -1 0, limit lower=0.0 upper=0.8 effort=50 velocity=0.5, mimic joint=robotiq_85_left_knuckle_joint
- added joint robotiq_85_right_inner_knuckle_joint: type revolute, parent robotiq_85_base_link, child robotiq_85_right_inner_knuckle_link, origin xyz=-0.0127 0.0 0.06142 rpy=0 0 0, axis 0 -1 0, limit lower=-0.8 upper=0.0 effort=50 velocity=0.5, mimic joint=robotiq_85_left_knuckle_joint multiplier=-1
- added joint robotiq_85_right_knuckle_joint: type revolute, parent robotiq_85_base_link, child robotiq_85_right_knuckle_link, origin xyz=-0.03060114 0.0 0.05490452 rpy=0 0 0, axis 0 -1 0, limit lower=-0.8 upper=0.0 effort=50 velocity=0.5, mimic joint=robotiq_85_left_knuckle_joint multiplier=-1
